Commit message: add torso model

File: gopher_description/torso_description/urdf/torso.urdf.xacro (robot description, xacro)
@@ -10,5 +10,5 @@
                 <origin xyz="0 0 ${height/2}" rpy="0 0 0"/>
                 <geometry>
-                    <box size="${width} ${width} ${height}"/>
+                    <mesh filename="package://gopher_description/torso_description/meshes/torso.dae" />
                 </geometry>
             </collision>
@@ -16,5 +16,5 @@
                 <origin xyz="0 0 ${height/2}" rpy="0 0 0"/>
                 <geometry>
-                    <box size="${width} ${width} ${height}"/>
+                    <mesh filename="package://gopher_description/torso_description/meshes/torso.dae" />
                 </geometry>
                 <material name="">
