Commit message: reorganize folder

File: gopher_description/realsense2_description/urdf/_d435.urdf.xacro (robot description, xacro)
@@ -8,5 +8,5 @@
 <robot name="sensor_d435" xmlns:xacro="http://ros.org/wiki/xacro">
   <!--File includes-->
-  <xacro:include filename="$(find gopher_description)/camera/urdf/_d435.gazebo.xacro"/>
+  <xacro:include filename="$(find gopher_description)/realsense2_description/urdf/_d435.gazebo.xacro"/>
   <xacro:macro name="sensor_d435" params="name:=camera prefix:=camera/ parent
                                           fov:=69.4 width:=1920 height:=1080
@@ -50,5 +50,5 @@
         <geometry>
           <!-- <box size="${d435_cam_width} ${d435_cam_height} ${d435_cam_depth}"/> -->
-          <mesh filename="package://gopher_description/camera/meshes/d435.dae" />
+          <mesh filename="package://gopher_description/realsense2_description/meshes/d435.dae" />
           <!--<mesh filename="package://realsense2_description/meshes/d435/d435.dae" />-->
         </geometry>

File: gopher_description/realsense2_description/urdf/arm_camera.urdf.xacro (robot description, xacro)
@@ -31,5 +31,5 @@
             <axis xyz="0 0 1"/>
         </joint>
-        <xacro:include filename="$(find gopher_description)/camera/urdf/_d435.urdf.xacro"/>
+        <xacro:include filename="$(find gopher_description)/realsense2_description/urdf/_d435.urdf.xacro"/>
         <xacro:sensor_d435 name="${camera_name}" prefix="${prefix}"
                            parent="${prefix}support"

File: gopher_description/realsense2_description/urdf/main_camera_support.urdf.xacro (robot description, xacro)
@@ -118,5 +118,5 @@
             </actuator>
         </transmission>
-        <xacro:include filename="$(find gopher_description)/camera/urdf/_d435.urdf.xacro"/>
+        <xacro:include filename="$(find gopher_description)/realsense2_description/urdf/_d435.urdf.xacro"/>
         <xacro:sensor_d435 name="${camera_name}" prefix="${prefix}"
                            parent="${prefix}pitch_link"

File: gopher_description/robots/urdf/gopher.xacro (robot description, xacro)
@@ -16,6 +16,6 @@
     <xacro:include filename="$(find gopher_description)/torso_description/urdf/torso.urdf.xacro" />
     <xacro:include filename="$(find gopher_description)/arms/urdf/kortex_robot.xacro" />
-    <xacro:include filename="$(find gopher_description)/camera/urdf/main_camera_support.urdf.xacro" />
-    <xacro:include filename="$(find gopher_description)/camera/urdf/arm_camera.urdf.xacro" />
+    <xacro:include filename="$(find gopher_description)/realsense2_description/urdf/main_camera_support.urdf.xacro" />
+    <xacro:include filename="$(find gopher_description)/realsense2_description/urdf/arm_camera.urdf.xacro" />
     <!-- Load the base -->
     <xacro:load_base prefix="$(arg prefix)"/>
