Commit message: rm parent link condition

File: gopher_description/kortex_description/arms/urdf/kortex_robot.xacro (robot description, xacro)
@@ -1,5 +1,5 @@
 <?xml version="1.0"?>
 <robot xmlns:xacro="http://ros.org/wiki/xacro">
-    <xacro:macro name="load_robot" params="arm gripper dof vision sim prefix parent">
+    <xacro:macro name="load_kortex" params="arm gripper dof vision sim prefix parent *origin">
         <!-- Files to include -->
         <xacro:include filename="$(find kortex_description)/arms/${arm}/${dof}dof/urdf/${arm}_macro.xacro" />
@@ -16,12 +16,10 @@
         </xacro:if>
         <!-- Run the macros -->
-        <!-- For gazebo -->
-        <xacro:if value="${sim}">
-            <joint name="${prefix}shoulder_to_arm_root" type="fixed">
-                <child link="${prefix}base_link" />
-                <parent link="${parent}" />
-                <origin xyz="0 0 0" rpy="0 0 0" />
-            </joint>
-        </xacro:if>
+        <!-- Attach to parent link -->
+        <joint name="${prefix}shoulder_to_arm_root" type="fixed">
+            <child link="${prefix}base_link" />
+            <parent link="${parent}" />
+            <xacro:insert_block name="origin" />
+        </joint>
         <!-- Load the arm -->
         <xacro:load_arm parent="" dof="${dof}" vision="${vision}" prefix="${prefix}">
@@ -43,5 +41,5 @@
             </joint>
         </xacro:if>
-        <!-- Load the Gazebo transmissions and gazebo_ros_control plugin -->
+        <!-- Load the Gazebo transmissions -->
         <xacro:if value="${sim}">
             <xacro:load_gazebo_arm_transmissions prefix="${prefix}"/>

File: gopher_description/robots/urdf/gopher.xacro (robot description, xacro)
@@ -29,7 +29,9 @@
     <xacro:if value="$(arg with_arms)">
         <!-- Load the right arm -->
-        <xacro:load_robot arm="$(arg arm)" gripper="$(arg gripper)" dof="$(arg dof)"
+        <xacro:load_kortex arm="$(arg arm)" gripper="$(arg gripper)" dof="$(arg dof)"
                           vision="$(arg vision)" sim="$(arg sim)"
-                          prefix="$(arg right_prefix)" parent="$(arg prefix)right_shoulder_link"/>
+                          prefix="$(arg right_prefix)" parent="$(arg prefix)right_shoulder_link">
+            <origin xyz="0 0 0" rpy="0 0 0" />
+        </xacro:load_kortex>
         <!-- Load arm camera -->
         <xacro:load_arm_camera prefix="$(arg right_prefix)cam_" camera_name="right_arm_cam"
@@ -37,7 +39,9 @@
                                width="1080" height="720" update_rate="30" wide_flag="true"/>
         <!-- Load the left arm -->
-        <xacro:load_robot arm="$(arg arm)" gripper="$(arg gripper)" dof="$(arg dof)"
+        <xacro:load_kortex arm="$(arg arm)" gripper="$(arg gripper)" dof="$(arg dof)"
                           vision="$(arg vision)" sim="$(arg sim)"
-                          prefix="$(arg left_prefix)" parent="$(arg prefix)left_shoulder_link"/>
+                          prefix="$(arg left_prefix)" parent="$(arg prefix)left_shoulder_link">
+            <origin xyz="0 0 0" rpy="0 0 0" />
+        </xacro:load_kortex>
         <!-- Load arm camera -->
         <xacro:load_arm_camera prefix="$(arg left_prefix)cam_" camera_name="left_arm_cam"
