Commit message: seperate gazebo urdf

File: gopher_description/robots/urdf/gopher.xacro (robot description, xacro)
@@ -15,4 +15,5 @@
     <xacro:include filename="$(find gopher_description)/fetch_description/urdf/freight_macro.xacro" />
     <xacro:include filename="$(find gopher_description)/torso_description/urdf/torso.urdf.xacro" />
+    <xacro:include filename="$(find gopher_description)/torso_description/urdf/torso.gazebo.xacro" />
     <xacro:include filename="$(find gopher_description)/kortex_description/arms/urdf/kortex_robot.xacro" />
     <xacro:include filename="$(find gopher_description)/realsense2_description/urdf/main_camera_support.urdf.xacro" />
@@ -21,16 +22,18 @@
     <xacro:load_base prefix="$(arg prefix)"/>
     <!-- Load torso -->
-    <xacro:load_torso prefix="$(arg prefix)"/>
-    <!-- Load main camera -->
+    <xacro:load_torso_urdf prefix="$(arg prefix)" parent="$(arg prefix)chassis_link"/>
+    <xacro:load_torso_gazebo prefix="$(arg prefix)"/>
+    <!-- Load main camera
     <xacro:load_main_camera prefix="$(arg prefix)main_cam_" camera_name="main_cam"
                             main_camera_base="$(arg prefix)torso"
                             width="1080" height="720" update_rate="30" wide_flag="true"/>
+    -->
     <!-- Load two arms -->
     <xacro:if value="$(arg with_arms)">
         <!-- Load the right arm -->
         <xacro:load_kortex arm="$(arg arm)" gripper="$(arg gripper)" dof="$(arg dof)"
-                          vision="$(arg vision)" sim="$(arg sim)"
-                          prefix="$(arg right_prefix)" parent="$(arg prefix)right_shoulder_link">
-            <origin xyz="0 0 0" rpy="0 0 0" />
+                           vision="$(arg vision)" sim="$(arg sim)"
+                           prefix="$(arg right_prefix)" parent="$(arg prefix)torso">
+            <origin xyz="-0.03 -0.03 0.7" rpy="1.5708 0 0" />
         </xacro:load_kortex>
         <!-- Load arm camera -->
@@ -40,7 +43,7 @@
         <!-- Load the left arm -->
         <xacro:load_kortex arm="$(arg arm)" gripper="$(arg gripper)" dof="$(arg dof)"
-                          vision="$(arg vision)" sim="$(arg sim)"
-                          prefix="$(arg left_prefix)" parent="$(arg prefix)left_shoulder_link">
-            <origin xyz="0 0 0" rpy="0 0 0" />
+                           vision="$(arg vision)" sim="$(arg sim)"
+                           prefix="$(arg left_prefix)" parent="$(arg prefix)torso">
+            <origin xyz="-0.03 0.03 0.7" rpy="1.5708 0 3.1416" />
         </xacro:load_kortex>
         <!-- Load arm camera -->

File: gopher_description/torso_description/urdf/torso.urdf.xacro (robot description, xacro)
@@ -1,93 +1,119 @@
 <?xml version="1.0"?>
 <robot name="robot_torso" xmlns:xacro="http://www.ros.org/wiki/xacro">
-    <xacro:macro name="load_torso" params="prefix">
-        <xacro:property name="mass" value="5.0" />
-        <xacro:property name="width" value="0.15" />
-        <xacro:property name="height" value="0.8" />
-        <xacro:property name="axel_offset" value="-0.25" />
-        <link name="${prefix}torso">
-            <collision>
-                <origin xyz="0 0 ${height/2}" rpy="0 0 0"/>
-                <geometry>
-                    <mesh filename="package://gopher_description/torso_description/meshes/torso.dae" />
-                </geometry>
-            </collision>
-            <visual>
-                <origin xyz="0 0 ${height/2}" rpy="0 0 0"/>
-                <geometry>
-                    <mesh filename="package://gopher_description/torso_description/meshes/torso.dae" />
-                </geometry>
-                <material name="">
-                    <color rgba="0.5 0.6 0.7 1"/>
-                </material>
-            </visual>
-            <inertial>
-                <origin xyz="0 0 ${height/2}" rpy="0 0 0"/>
-                <mass value="${mass}"/>
-                <inertia ixx="${mass / 12.0 * (width*width + height*height)}" ixy="0.0" ixz="0.0"
-                        iyy="${mass / 12.0 * (height*height + width*width)}" iyz="0.0"
-                        izz="${mass / 12.0 * (width*width + width*width)}"/>
-            </inertial>
-        </link>
-        <joint name="${prefix}torso_joint" type="fixed">
-            <parent link="${prefix}chassis_link"/>
-            <child link="${prefix}torso"/>
-            <origin xyz="-0.0 0 0.36" rpy="0 0 0"/>
-            <axis xyz="0 0 1"/>
-        </joint>
-        <link name="${prefix}right_shoulder_link">
-            <collision>
-            <origin xyz="0 0 0" rpy="0 0 0"/>
-            <geometry>
-                <box size="0.001 0.001 0.001"/>
-            </geometry>
-            </collision>
-            <visual>
-            <origin xyz="0 0 0" rpy="0 0 0"/>
-            <geometry>
-                <box size="0.001 0.001 0.001"/>
-            </geometry>
-            </visual>
-            <inertial>
-            <origin xyz="0 0 0" rpy="0 0 0"/>
-            <mass value="0.0"/>
-            <inertia ixx="0.01" ixy="0.01" ixz="0.01"
-                     iyy="0.01" iyz="0.01"
-                     izz="0.01"/>
-            </inertial>
-        </link>
-        <joint name="${prefix}right_shoulder_to_torso_joint" type="fixed">
-            <child link="${prefix}right_shoulder_link" />
-            <parent link="${prefix}torso" />
-            <origin xyz="0 0 0.7" rpy="1.57 0 0" />
-            <axis xyz="0 0 1"/>
-        </joint>
-        <link name="${prefix}left_shoulder_link">
-            <collision>
-            <origin xyz="0 0 0" rpy="0 0 0"/>
-            <geometry>
-                <box size="0.001 0.001 0.001"/>
-            </geometry>
-            </collision>
-            <visual>
-            <origin xyz="0 0 0" rpy="0 0 0"/>
-            <geometry>
-                <box size="0.001 0.001 0.001"/>
-            </geometry>
-            </visual>
-            <inertial>
-            <origin xyz="0 0 0" rpy="0 0 0"/>
-            <mass value="0.0"/>
-            <inertia ixx="0.01" ixy="0.01" ixz="0.01"
-                     iyy="0.01" iyz="0.01"
-                     izz="0.01"/>
-            </inertial>
-        </link>
-        <joint name="${prefix}left_shoulder_to_torso_joint" type="fixed">
-            <child link="${prefix}left_shoulder_link" />
-            <parent link="${prefix}torso" />
-            <origin xyz="0 0 0.7" rpy="-1.57 0 0" />
-            <axis xyz="0 0 1"/>
-        </joint>
+  <xacro:macro name="load_torso_urdf" params="prefix parent">
+    <link name="${prefix}torso">
+      <inertial>
+        <origin rpy="0 0 0" xyz="0.0 0.0 0.4" />
+        <mass value="12.0" />
+        <inertia ixx="0.68" ixy="0.0" ixz="0.0" iyy="0.73" iyz="0.0" izz="0.13" />
+      </inertial>
+      <visual>
+        <origin rpy="0 0 0" xyz="0 0 0" />
+        <geometry>
+          <mesh filename="package://gopher_description/torso_description/meshes/torso.dae" />
+        </geometry>
+        <material name="">
+          <color rgba="0.3 0.3 0.3 1" />
+        </material>
+      </visual>
+      <collision>
+        <origin rpy="0 0 0" xyz="0 0 0" />
+        <geometry>
+          <mesh filename="package://gopher_description/torso_description/meshes/torso.dae" />
+        </geometry>
+      </collision>
+    </link>
+    <joint name="${prefix}torso_joint" type="fixed">
+      <parent link="${parent}"/>
+      <child link="${prefix}torso"/>
+      <origin xyz="-0.0 0 0.36" rpy="0 0 0"/>
+      <axis xyz="0 0 1"/>
+    </joint>
+    <link name="${prefix}main_cam_support">
+      <collision>
+        <origin rpy="0 0 0" xyz="0 0 0.01"/>
+        <geometry>
+          <box size="0.08 0.08 0.02"/>
+        </geometry>
+      </collision>
+      <visual>
+        <origin rpy="0 0 0" xyz="0 0 0.01"/>
+        <geometry>
+          <box size="0.08 0.08 0.02"/>
+        </geometry>
+        <material name="">
+          <color rgba="0.5 0.6 0.7 1"/>
+        </material>
+      </visual>
+      <inertial>
+        <origin rpy="0 0 0" xyz="0 0 0.01"/>
+        <mass value="0.36"/>
+        <inertia ixx="2.04e-04" ixy="0.0" ixz="0.0" iyy="2.04e-04" iyz="0.0" izz="3.84e-04"/>
+      </inertial>
+    </link>
+    <joint name="${prefix}main_cam_support_joint" type="fixed">
+      <parent link="${prefix}torso"/>
+      <child link="${prefix}main_cam_support"/>
+      <origin rpy="0 0 0" xyz="0.0 0.0 0.8"/>
+      <axis xyz="0 0 1"/>
+    </joint>
+    <link name="${prefix}main_cam_yaw_link">
+      <collision>
+        <origin rpy="0 0 0" xyz="0 0 0.03"/>
+        <geometry>
+          <box size="0.03 0.03 0.06"/>
+        </geometry>
+      </collision>
+      <visual>
+        <origin rpy="0 0 0" xyz="0 0 0.03"/>
+        <geometry>
+          <box size="0.03 0.03 0.06"/>
+        </geometry>
+        <material name="blue">
+          <color rgba="0 0 1 1"/>
+        </material>
+      </visual>
+      <inertial>
+        <origin rpy="0 0 0" xyz="0 0 0.03"/>
+        <mass value="0.36"/>
+        <inertia ixx="1.35e-01" ixy="0.0" ixz="0.0" iyy="1.35e-01" iyz="0.0" izz="5.4e-02"/>
+      </inertial>
+    </link>
+    <joint name="${prefix}main_cam_yaw_joint" type="revolute">
+      <parent link="${prefix}main_cam_support"/>
+      <child link="${prefix}main_cam_yaw_link"/>
+      <origin rpy="0 0 0" xyz="0 0 0.02"/>
+      <axis xyz="0 0 1"/>
+      <limit effort="20" lower="-1.047" upper="1.047" velocity="1.0"/>
+    </joint>
+    <link name="${prefix}main_cam_pitch_link">
+      <collision>
+        <origin rpy="0 1.5708 0" xyz="0.03 0 0"/>
+        <geometry>
+          <box size="0.03 0.03 0.06"/>
+        </geometry>
+      </collision>
+      <visual>
+        <origin rpy="0 1.5708 0" xyz="0.03 0 0"/>
+        <geometry>
+          <box size="0.03 0.03 0.06"/>
+        </geometry>
+        <material name="red">
+          <color rgba="1 0 0 1"/>
+        </material>
+      </visual>
+      <inertial>
+        <origin rpy="0 1.5708 0" xyz="0.03 0 0"/>
+        <mass value="0.36"/>
+        <inertia ixx="1.35e-01" ixy="0.0" ixz="0.0" iyy="1.35e-01" iyz="0.0" izz="5.4e-02"/>
+      </inertial>
+    </link>
+    <joint name="${prefix}main_cam_pitch_joint" type="revolute">
+      <parent link="${prefix}main_cam_yaw_link"/>
+      <child link="${prefix}main_cam_pitch_link"/>
+      <origin rpy="1.5708 0 0" xyz="0.0 0.0 0.06"/>
+      <axis xyz="0 0 1"/>
+      <limit effort="20" lower="-1.047" upper="1.047" velocity="1.0"/>
+    </joint>
     </xacro:macro>
 </robot>
