Commit message: seperate gazebo urdf

File: gopher_description/fetch_description/urdf/freight.gazebo.xacro (robot description, xacro)
@@ -1,8 +1,5 @@
 <?xml version="1.0"?>
 <robot name="freight" xmlns:xacro="http://www.ros.org/wiki/xacro">
-  <xacro:macro name="load_base" params="prefix">
-      <!-- <xacro:include filename="$(find fetch_description)/robots/freight.urdf.xacro" /> -->
-      <xacro:include filename="$(find gopher_description)/fetch_description/urdf/freight.urdf.xacro" />
-      <xacro:load_base_urdf prefix="${prefix}"/>
+  <xacro:macro name="load_freight_gazebo" params="prefix">
       <!-- Base is modeled as a big tub sitting on floor, with two wheels -->
       <gazebo reference="${prefix}chassis_link">
@@ -26,8 +23,4 @@
         <material>Gazebo/Black</material>
       </gazebo>
-      <!-- Color the estop -->
-      <gazebo reference="${prefix}estop_link">
-        <material>Gazebo/Red</material>
-      </gazebo>
       <gazebo reference="${prefix}l_wheel_joint">
         <implicitSpringDamper>1</implicitSpringDamper>
@@ -35,7 +28,4 @@
       <gazebo reference="${prefix}r_wheel_joint">
         <implicitSpringDamper>1</implicitSpringDamper>
-      </gazebo>
-      <gazebo reference="${prefix}camera_support">
-        <material>Gazebo/Black</material>
       </gazebo>
       <!-- SICK TIM561 (25m Range) -->
@@ -73,4 +63,27 @@
         </sensor>
       </gazebo>
+      <!-- Color the estop -->
+      <gazebo reference="${prefix}estop_link">
+        <material>Gazebo/Red</material>
+      </gazebo>
+      <!-- Transmission -->
+      <transmission name="${prefix}r_wheel_trans">
+      <type>transmission_interface/SimpleTransmission</type>
+      <joint name="${prefix}r_wheel_joint">
+          <hardwareInterface>hardware_interface/VelocityJointInterface</hardwareInterface>
+      </joint>
+      <actuator name="${prefix}r_wheel_actuator">
+          <mechanicalReduction>1</mechanicalReduction>
+      </actuator>
+    </transmission>
+    <transmission name="${prefix}l_wheel_trans">
+      <type>transmission_interface/SimpleTransmission</type>
+      <joint name="${prefix}l_wheel_joint">
+          <hardwareInterface>hardware_interface/VelocityJointInterface</hardwareInterface>
+      </joint>
+      <actuator name="${prefix}l_wheel_actuator">
+          <mechanicalReduction>1</mechanicalReduction>
+      </actuator>
+    </transmission>
   </xacro:macro>
 </robot>

File: gopher_description/fetch_description/urdf/freight.urdf.xacro (robot description, xacro)
@@ -1,11 +1,6 @@
 <?xml version="1.0"?>
 <robot name="freight" xmlns:xacro="http://www.ros.org/wiki/xacro">
-  <xacro:macro name="load_base_urdf" params="prefix">
-    <link name="${prefix}base_link"></link>
-    <joint name="${prefix}base_link_joint" type="fixed">
-        <origin xyz="0 0 0" rpy="0 0 0" />
-        <parent link="${prefix}base_link"/>
-        <child link="${prefix}chassis_link" />
-    </joint>
+  <xacro:macro name="load_freight_urdf" params="prefix">
+    <link name="${prefix}base_link"/>
     <link name="${prefix}chassis_link">
       <inertial>
@@ -19,7 +14,4 @@
           <mesh filename="package://gopher_description/fetch_description/meshes/base_link.dae" />
         </geometry>
-        <material name="">
-          <color rgba="0.356 0.361 0.376 1" />
-        </material>
       </visual>
       <collision>
@@ -30,4 +22,8 @@
       </collision>
     </link>
+    <joint name="${prefix}base_joint" type="fixed">
+      <parent link="${prefix}base_link"/>
+      <child link="${prefix}chassis_link"/>
+    </joint>
     <link name="${prefix}r_wheel_link">
       <inertial>
@@ -53,6 +49,5 @@
     </link>
     <joint name="${prefix}r_wheel_joint" type="continuous">
-      <!--origin rpy="-6.123E-17 0 0" xyz="0.0012914 -0.18738 0.055325" -->
-      <origin rpy="-6.123E-17 0 0" xyz="0.0012914 -0.18738 0.0602" />
+      <origin rpy="-6.123E-17 0 0" xyz="0.0012914 -0.18738 0.0602" /> <!-- r 0.0605 -->
       <parent link="${prefix}chassis_link" />
       <child link="${prefix}r_wheel_link" />
@@ -83,6 +78,5 @@
     </link>
     <joint name="${prefix}l_wheel_joint" type="continuous">
-      <!-- origin rpy="-6.123E-17 0 0" xyz="0.0012914 0.18738 0.055325" -->
-      <origin rpy="-6.123E-17 0 0" xyz="0.0012914 0.18738 0.0602" />
+      <origin rpy="-6.123E-17 0 0" xyz="0.0012914 0.18738 0.0602" /> <!-- r 0.0605 -->
       <parent link="${prefix}chassis_link" />
       <child link="${prefix}l_wheel_link" />
@@ -158,22 +152,4 @@
       <child link="${prefix}base_camera_optical_frame" />
     </joint>
-    <transmission name="${prefix}r_wheel_trans">
-      <type>transmission_interface/SimpleTransmission</type>
-      <joint name="${prefix}r_wheel_joint">
-          <hardwareInterface>hardware_interface/VelocityJointInterface</hardwareInterface>
-      </joint>
-      <actuator name="${prefix}r_wheel_actuator">
-          <mechanicalReduction>1</mechanicalReduction>
-      </actuator>
-    </transmission>
-    <transmission name="${prefix}l_wheel_trans">
-      <type>transmission_interface/SimpleTransmission</type>
-      <joint name="${prefix}l_wheel_joint">
-          <hardwareInterface>hardware_interface/VelocityJointInterface</hardwareInterface>
-      </joint>
-      <actuator name="${prefix}l_wheel_actuator">
-          <mechanicalReduction>1</mechanicalReduction>
-      </actuator>
-    </transmission>
   </xacro:macro>
 </robot>

File: gopher_description/realsense2_description/urdf/_d435.gazebo.xacro (robot description, xacro)
@@ -5,9 +5,6 @@
 -->
 <robot xmlns:xacro="http://ros.org/wiki/xacro">
-  <xacro:macro name="gazebo_d435" params="camera_name reference_link
-                                          color_optical_frame
-                                          fov:=69.4 width:=1920 height:=1080
-                                          update_rate:=30" >
-    <!-- Load parameters to model's main link-->
+  <xacro:macro name="gazebo_d435" params="camera_name reference_link frame_name
+                                          fov:=69.4 width:=1920 height:=1080 update_rate:=30" >
     <xacro:property name="deg_to_rad" value="0.01745329251994329577" />
     <gazebo reference="${reference_link}">
@@ -28,22 +25,22 @@
           </clip>
         </camera>
-        <plugin name="${camera_name}_controller" filename="libgazebo_ros_openni_kinect.so">
+        <plugin name="${camera_name}_plugin" filename="libgazebo_ros_openni_kinect.so">
           <baseline>0.2</baseline>
           <alwaysOn>true</alwaysOn>
           <updateRate>0.0</updateRate>
           <cameraName>${camera_name}</cameraName>
-          <frameName>${color_optical_frame}</frameName>
           <imageTopicName>color/image_raw</imageTopicName>
+          <cameraInfoTopicName>color/camera_info</cameraInfoTopicName>
           <depthImageTopicName>depth/image_raw</depthImageTopicName>
+          <depthImageCameraInfoTopicName>depth/camera_info</depthImageCameraInfoTopicName>
           <pointCloudTopicName>depth/points</pointCloudTopicName>
-          <cameraInfoTopicName>color/camera_info</cameraInfoTopicName>
-          <depthImageCameraInfoTopicName>depth/camera_info</depthImageCameraInfoTopicName>
+          <frameName>${frame_name}</frameName>
           <pointCloudCutoff>0.5</pointCloudCutoff>
           <pointCloudCutoffMax>3.0</pointCloudCutoffMax>
-          <distortionK1>0</distortionK1>
-          <distortionK2>0</distortionK2>
-          <distortionK3>0</distortionK3>
-          <distortionT1>0</distortionT1>
-          <distortionT2>0</distortionT2>
+          <distortionK1>0.00000001</distortionK1>
+          <distortionK2>0.00000001</distortionK2>
+          <distortionK3>0.00000001</distortionK3>
+          <distortionT1>0.00000001</distortionT1>
+          <distortionT2>0.00000001</distortionT2>
           <CxPrime>0</CxPrime>
           <Cx>0</Cx>

File: gopher_description/realsense2_description/urdf/_d435.urdf.xacro (robot description, xacro)
@@ -7,9 +7,5 @@
 -->
 <robot name="sensor_d435" xmlns:xacro="http://ros.org/wiki/xacro">
-  <!--File includes-->
-  <xacro:include filename="$(find gopher_description)/realsense2_description/urdf/_d435.gazebo.xacro"/>
-  <xacro:macro name="sensor_d435" params="name:=camera prefix:=camera/ parent
-                                          fov:=69.4 width:=1920 height:=1080
-                                          update_rate:=60 wide_flag:=false *origin">
+  <xacro:macro name="sensor_d435" params="prefix parent *origin">
     <xacro:property name="M_PI" value="3.1415926535897931" />
     <!-- The following values are approximate, and the camera node
@@ -30,6 +26,6 @@
     <xacro:property name="d435_cam_depth_py" value="0.0175"/>
     <xacro:property name="d435_cam_depth_pz" value="${d435_cam_height/2}"/>
-    <material name="${prefix}aluminum">
-	  <color rgba="0.5 0.5 0.5 1"/>
+    <material name="aluminum">
+	    <color rgba="0.5 0.5 0.5 1"/>
     </material>
     <!-- camera body, with origin at bottom screw mount -->
@@ -49,14 +45,12 @@
       <origin xyz="${d435_cam_mount_from_center_offset} ${-d435_cam_depth_py} 0" rpy="${M_PI/2} 0 ${M_PI/2}"/>
         <geometry>
-          <!-- <box size="${d435_cam_width} ${d435_cam_height} ${d435_cam_depth}"/> -->
           <mesh filename="package://gopher_description/realsense2_description/meshes/d435.dae" />
-          <!--<mesh filename="package://realsense2_description/meshes/d435/d435.dae" />-->
         </geometry>
-        <material name="${prefix}aluminum"/>
+        <material name="aluminum"/>
       </visual>
       <collision>
         <origin xyz="0 ${-d435_cam_depth_py} 0" rpy="0 0 0"/>
         <geometry>
-        <box size="${d435_cam_depth} ${d435_cam_width} ${d435_cam_height}"/>
+          <box size="${d435_cam_depth} ${d435_cam_width} ${d435_cam_height}"/>
         </geometry>
       </collision>
@@ -122,17 +116,4 @@
     </joint>
     <link name="${prefix}color_optical_frame"/>
-    <!-- Realsense Gazebo Plugin -->
-    <!-- Normal camera -->
-    <xacro:gazebo_d435 camera_name="${name}" reference_link="${prefix}link"
-                      color_optical_frame="${name}_color_optical_frame"
-                      fov="${fov}" width="${width}" height="${height}"
-                      update_rate="${update_rate}"/>
-    <!-- Wide camera -->
-    <xacro:if value="${wide_flag}">
-    <xacro:gazebo_d435 camera_name="${name}_wide" reference_link="${prefix}link"
-                      color_optical_frame="${name}_color_optical_frame"
-                      fov="114" width="${1.5555*width}" height="${height}"
-                      update_rate="${update_rate}"/>
-    </xacro:if>
   </xacro:macro>
 </robot>

File: gopher_description/robots/urdf/gopher.xacro (robot description, xacro)
@@ -11,25 +11,22 @@
     <xacro:arg name="dof" default="7" />
     <xacro:arg name="vision" default="true" />
-    <xacro:arg name="sim" default="true" />
+    <!-- Simulate in gazebo -->
+    <xacro:arg name="sim" default="true" />b
     <!-- Include files -->
-    <xacro:include filename="$(find gopher_description)/fetch_description/urdf/freight_macro.xacro" />
+    <xacro:include filename="$(find gopher_description)/fetch_description/urdf/freight.urdf.xacro" />
     <xacro:include filename="$(find gopher_description)/torso_description/urdf/torso.urdf.xacro" />
-    <xacro:include filename="$(find gopher_description)/torso_description/urdf/torso.gazebo.xacro" />
+    <xacro:include filename="$(find gopher_description)/realsense2_description/urdf/_d435.urdf.xacro" />
     <xacro:include filename="$(find gopher_description)/kortex_description/arms/urdf/kortex_robot.xacro" />
-    <xacro:include filename="$(find gopher_description)/realsense2_description/urdf/main_camera_support.urdf.xacro" />
-    <xacro:include filename="$(find gopher_description)/realsense2_description/urdf/arm_camera.urdf.xacro" />
-    <!-- Load the base -->
-    <xacro:load_base prefix="$(arg prefix)"/>
-    <!-- Load torso -->
-    <xacro:load_torso_urdf prefix="$(arg prefix)" parent="$(arg prefix)chassis_link"/>
-    <xacro:load_torso_gazebo prefix="$(arg prefix)"/>
-    <!-- Load main camera
-    <xacro:load_main_camera prefix="$(arg prefix)main_cam_" camera_name="main_cam"
-                            main_camera_base="$(arg prefix)torso"
-                            width="1080" height="720" update_rate="30" wide_flag="true"/>
-    -->
-    <!-- Load two arms -->
+    <!-- Load urdf -->
+    <!-- base -->
+    <xacro:load_freight_urdf prefix="$(arg prefix)" />
+    <!-- torso -->
+    <xacro:load_torso_urdf prefix="$(arg prefix)" parent="$(arg prefix)chassis_link" />
+    <!-- main camera -->
+    <xacro:sensor_d435 prefix="$(arg prefix)main_cam_" parent="$(arg prefix)main_cam_pitch_link">
+        <origin xyz="0.06 -0.01 0.0" rpy="-1.57 0 0" />
+    </xacro:sensor_d435>
+    <!-- arms -->
     <xacro:if value="$(arg with_arms)">
-        <!-- Load the right arm -->
         <xacro:load_kortex arm="$(arg arm)" gripper="$(arg gripper)" dof="$(arg dof)"
                            vision="$(arg vision)" sim="$(arg sim)"
@@ -37,9 +34,4 @@
             <origin xyz="-0.03 -0.03 0.7" rpy="1.5708 0 0" />
         </xacro:load_kortex>
-        <!-- Load arm camera -->
-        <xacro:load_arm_camera prefix="$(arg right_prefix)cam_" camera_name="right_arm_cam"
-                               arm_camera_base="$(arg right_prefix)camera_link"
-                               width="1080" height="720" update_rate="30" wide_flag="true"/>
-        <!-- Load the left arm -->
         <xacro:load_kortex arm="$(arg arm)" gripper="$(arg gripper)" dof="$(arg dof)"
                            vision="$(arg vision)" sim="$(arg sim)"
@@ -47,14 +39,43 @@
             <origin xyz="-0.03 0.03 0.7" rpy="1.5708 0 3.1416" />
         </xacro:load_kortex>
-        <!-- Load arm camera -->
-        <xacro:load_arm_camera prefix="$(arg left_prefix)cam_" camera_name="left_arm_cam"
-                               arm_camera_base="$(arg left_prefix)camera_link"
-                               width="1080" height="720" update_rate="30" wide_flag="true"/>
     </xacro:if>
-    <!-- Load gazebo control pulgin ONLY ONCE -->
-    <gazebo>
-        <plugin name="gazebo_ros_control" filename="libgazebo_ros_control.so">
-            <legacyModeNS>true</legacyModeNS>
-        </plugin>
-    </gazebo>
+    <!-- Load gazebo control pulgin -->
+    <xacro:if value="$(arg sim)">
+        <xacro:include filename="$(find gopher_description)/fetch_description/urdf/freight.gazebo.xacro" />
+        <xacro:include filename="$(find gopher_description)/torso_description/urdf/torso.gazebo.xacro" />
+        <xacro:include filename="$(find gopher_description)/realsense2_description/urdf/_d435.gazebo.xacro" />
+        <xacro:load_freight_gazebo prefix="$(arg prefix)" />
+        <xacro:load_torso_gazebo prefix="$(arg prefix)" />
+        <xacro:gazebo_d435 camera_name="main_cam" reference_link="$(arg prefix)main_cam_link"
+                           frame_name="main_cam_color_optical_frame"
+                           fov="69.4" width="1080" height="720" update_rate="30" />
+        <xacro:if value="$(arg with_arms)">
+            <link name="$(arg left_prefix)cam_link" />
+            <link name="$(arg right_prefix)cam_link" />
+            <joint name="$(arg left_prefix)cam_joint" type="fixed">
+                <origin xyz="0 0 0" rpy="0 -1.5709 1.5709" />
+                <parent link="$(arg left_prefix)camera_link" />
+                <child link="$(arg left_prefix)cam_link" />
+            </joint>
+            <joint name="$(arg right_prefix)cam_joint" type="fixed">
+                <origin xyz="0 0 0" rpy="0 -1.5709 1.5709" />
+                <parent link="$(arg right_prefix)camera_link" />
+                <child link="$(arg right_prefix)cam_link" />
+            </joint>
+            <xacro:gazebo_d435 camera_name="left_arm_cam" reference_link="$(arg left_prefix)cam_link"
+                            frame_name="left_arm_camera_color_frame"
+                            fov="69.4" width="1080" height="720" update_rate="30" />
+            <xacro:gazebo_d435 camera_name="right_arm_cam" reference_link="$(arg right_prefix)cam_link"
+                            frame_name="right_arm_camera_color_frame"
+                            fov="69.4" width="1080" height="720" update_rate="30" />
+            <!-- Wide FOV camera setting
+            fov="114" width="1.5555*1080" height="720" update_rate="30"
+            -->
+        </xacro:if>
+        <gazebo>
+            <plugin name="gazebo_ros_control" filename="libgazebo_ros_control.so">
+                <legacyModeNS>true</legacyModeNS>
+            </plugin>
+        </gazebo>
+    </xacro:if>
 </robot>
